Commit message: adding separate rsp launch file and updating xacro description

File: src/clyde_description/src/urdf/clyde_simple.xacro (robot description, xacro)
@@ -955,5 +955,5 @@
 </joint>
 <joint name="shrfs_joint" type="continuous">
-  <origin xyz="-0.007145 -0.0125 0.004125" rpy="0 0 0"/>
+  <origin xyz="-0.007145 -0.0125 0.004125" rpy="0 -1.308 0"/>
   <parent link="servo_rfs_1"/>
   <child link="c_thrf__1"/>
@@ -966,5 +966,5 @@
 </joint>
 <joint name="shrft_joint" type="continuous">
-  <origin xyz="0.0 0.007857 0.0" rpy="0 0 0"/>
+  <origin xyz="0.0 0.007857 0.0" rpy="0 1.206 0"/>
   <parent link="c_thorf_1"/>
   <child link="servos_rf_1"/>
@@ -997,5 +997,5 @@
 </joint>
 <joint name="shrrs_joint" type="continuous">
-  <origin xyz="0.007145 -0.0125 0.004125" rpy="0 0 0"/>
+  <origin xyz="0.007145 -0.0125 0.004125" rpy="0 -1.341 0"/>
   <parent link="servo_rrs__1"/>
   <child link="c_thrr_1"/>
@@ -1003,5 +1003,5 @@
 </joint>
 <joint name="shrrt_joint" type="continuous">
-  <origin xyz="0.0 0.007857 0.0" rpy="0 0 0"/>
+  <origin xyz="0.0 0.007857 0.0" rpy="0 1.206 0"/>
   <parent link="c_thorr_1"/>
   <child link="servos_rr_1"/>
@@ -1034,5 +1034,5 @@
 </joint>
 <joint name="shlfs_joint" type="continuous">
-  <origin xyz="-0.007145 0.0125 0.004125" rpy="0 0 0"/>
+  <origin xyz="-0.007145 0.0125 0.004125" rpy="0 -1.274 0"/>
   <parent link="servo_lfs_1"/>
   <child link="c_thlf_1"/>
@@ -1040,5 +1040,5 @@
 </joint>
 <joint name="shlft_joint" type="continuous">
-  <origin xyz="0.0 -0.007857 0.0" rpy="0 0 0"/>
+  <origin xyz="0.0 -0.007857 0.0" rpy="0 1.206 0"/>
   <parent link="c_tholf_1"/>
   <child link="servos_lf_1"/>
@@ -1071,5 +1071,5 @@
 </joint>
 <joint name="shlrs_joint" type="continuous">
-  <origin xyz="0.007145 0.0125 0.004125" rpy="0 0 0"/>
+  <origin xyz="0.007145 0.0125 0.004125" rpy="0 -1.308 0"/>
   <parent link="servo_lrs__1"/>
   <child link="c_thlr_1"/>
@@ -1077,5 +1077,5 @@
 </joint>
 <joint name="shlrt_joint" type="continuous">
-  <origin xyz="0.0 -0.007857 0.0" rpy="0 0 0"/>
+  <origin xyz="0.0 -0.007857 0.0" rpy="0 1.206 0"/>
   <parent link="c_tholr__1"/>
   <child link="servos_lr_1"/>
