Commit message: updating urdf to be same as real clyde

File: src/clyde_description/src/urdf/clyde_simple.urdf (robot description, URDF)
Before this commit: robot clyde, 45 links, 44 joints
Joints:
- joint shlfs_joint: origin xyz=-0.007145 0.0125 0.004125 rpy=0 0 0 -> xyz=-0.007145 0.0125 0.004125 rpy=0 -1.274 0
- joint shlft_joint: origin xyz=0.0 -0.007857 0.0 rpy=0 0 0 -> xyz=0.0 -0.007857 0.0 rpy=0 1.206 0
- joint shlrs_joint: origin xyz=0.007145 0.0125 0.004125 rpy=0 0 0 -> xyz=0.007145 0.0125 0.004125 rpy=0 -1.308 0
- joint shlrt_joint: origin xyz=0.0 -0.007857 0.0 rpy=0 0 0 -> xyz=0.0 -0.007857 0.0 rpy=0 1.206 0
- joint shrfs_joint: origin xyz=-0.007145 -0.0125 0.004125 rpy=0 0 0 -> xyz=-0.007145 -0.0125 0.004125 rpy=0 -1.308 0
- joint shrft_joint: origin xyz=0.0 0.007857 0.0 rpy=0 0 0 -> xyz=0.0 0.007857 0.0 rpy=0 1.206 0
- joint shrrs_joint: origin xyz=0.007145 -0.0125 0.004125 rpy=0 0 0 -> xyz=0.007145 -0.0125 0.004125 rpy=0 -1.341 0
- joint shrrt_joint: origin xyz=0.0 0.007857 0.0 rpy=0 0 0 -> xyz=0.0 0.007857 0.0 rpy=0 1.206 0

Commit message: robot state publisher script updated with urdf

File: src/clyde_description/src/urdf/clyde_simple.urdf (robot description, URDF)
Before this commit: robot clyde, 45 links, 44 joints
Joints:
- joint shlrs_joint: axis -0.0 -1.0 0.0 -> 0.0 1.0 0.0
- joint shrrs_joint: axis 0.0 -1.0 -0.0 -> 0.0 1.0 0.0

File: src/clyde_description/src/urdf/clyde_simple.xacro (robot description, xacro)
@@ -1000,5 +1000,5 @@
   <parent link="servo_rrs__1"/>
   <child link="c_thrr_1"/>
-  <axis xyz="0.0 -1.0 -0.0"/>
+  <axis xyz="0.0 1.0 0.0"/>
 </joint>
 <joint name="shrrt_joint" type="continuous">
@@ -1074,5 +1074,5 @@
   <parent link="servo_lrs__1"/>
   <child link="c_thlr_1"/>
-  <axis xyz="-0.0 -1.0 0.0"/>
+  <axis xyz="0.0 1.0 0.0"/>
 </joint>
 <joint name="shlrt_joint" type="continuous">
